File: HABs.kicad_pcb (KiCad board)
At the start: 0 parts

Commit message: feat: initial schematic
Parts:
- added A1: RaspberryPi_Pico, Module:RaspberryPi_Pico_Common_Unspecified, F.Cu at (114.3, 81.4)
- added IC1: CAM-M8C-0-10, CamM8C:CAMM8C010, F.Cu at (135.3, 59.0)
- added U2: Ai-Thinker-Ra-02, RF_Module:Ai-Thinker-Ra-01-LoRa, F.Cu at (136.2, 42.7)
Other:
- copper layers 0 -> 2
