File: HABs.kicad_sch (KiCad schematic)
At the start: 5 parts, among them IC1 CAM-M8C-0-10, J1 Conn_Coaxial, J2 Conn_01x02_Pin, U2 Ai-Thinker-Ra-02

Commit message: feat: initial schematic
Parts:
- removed J1: Conn_Coaxial, symbol Connector:Conn_Coaxial
- added J1: Conn_01x08_Pin, symbol Connector:Conn_01x08_Pin
- added U1: ~, symbol Components:MicroSD
- added U3: BMP180, symbol Components:BMP180
Connections:
- net GND: now also J1.1 (Pin_1), U1.6 (GND), U3.2 (GND)
- net LORA_BUSY: now also A1.26 (GPIO20); no longer A1.21 (GPIO16)
- net LORA_CS: now also A1.22 (GPIO17); no longer A1.27 (GPIO21)
- net LORA_MISO: now also A1.21 (GPIO16); no longer A1.25 (GPIO19)
- net LORA_MOSI: now also A1.25 (GPIO19); no longer A1.26 (GPIO20)
- net LORA_RESET: now also A1.27 (GPIO21); no longer A1.22 (GPIO17)
- net SCL: now also A1.10 (GPIO7), J1.2 (Pin_2); no longer A1.15 (GPIO11), IC1.6 (SCL_/_SPI_CLK)
- net SDA: now also A1.9 (GPIO6), J1.3 (Pin_3); no longer A1.14 (GPIO10), IC1.3 (SDA_/_SPI_CS_N)
- net BMP_SDA: now reaches A1.1 (GPIO0)
- net BMP_SDA: now also U3.4 (SDA)
- net SD_MISO: now reaches A1.11 (GPIO8)
- net SD_MISO: now also U1.5 (MISO)
- net SD_CS: now reaches A1.12 (GPIO9)
- net SD_CS: now also U1.2 (CS)
- net GPS_SDA: now reaches A1.19 (GPIO14)
- net GPS_SDA: now also IC1.3 (SDA_/_SPI_CS_N)
- net BMP_SCL: now reaches A1.2 (GPIO1)
- net BMP_SCL: now also U3.3 (SCL)
- net GPS_SCL: now reaches A1.20 (GPIO15)
- net GPS_SCL: now also IC1.6 (SCL_/_SPI_CLK)
- net SCK: now reaches A1.4 (GPIO2)
- net SCK: now also J1.7 (Pin_7)
- net MOSI: now reaches A1.5 (GPIO3)
- net MOSI: now also J1.6 (Pin_6)
- net MISO: now reaches A1.6 (GPIO4)
- net MISO: now also J1.5 (Pin_5)
- net CS: now reaches A1.7 (GPIO5)
- net CS: now also J1.4 (Pin_4)
- net 3.3V renamed +3.3V
- net +3.3V: now also J1.8 (Pin_8), U1.1 (3v3), U3.1 (VIN)
- net RX renamed GPS_RX
- net TX renamed GPS_TX
- new net SD_CLK: U1.4 (CLK)
- new net SD_MOSI: A1.15 (GPIO11), U1.3 (MOSI)
- new net SD_SCK: A1.14 (GPIO10)
- no-connect marks 13 -> 22
Other:
- note added: "BMP180/280 Temperature/Pressure"
- note added: "Breakout"
- note added: "GPS"
- note added: "LoRa"
- note added: "Micro SD"
- note added: "Power Input"
- note added: "RPI Pico"
- moved on the sheet: A1, IC1, J2, U2

Commit message: feat: initial PCB layout
Parts:
- added SW1: SW_SPDT, Button_Switch_THT:SW_Slide_SPDT_Angled_CK_OS102011MA1Q, symbol Switch:SW_SPDT
- J1: footprint (none) -> Connector_PinSocket_2.54mm:PinSocket_1x08_P2.54mm_Vertical
- J2: footprint (none) -> Connector_PinSocket_2.54mm:PinSocket_1x02_P2.54mm_Vertical
- U1: value ~ -> MicroSD; footprint (none) -> Components:MicroSD
- U3: footprint (none) -> Components:BMP180
Connections:
- net SD_SCK is gone; now on net SD_CLK: A1.14 (GPIO10)
- net VCC: now also SW1.1 (A); no longer J2.1 (Pin_1)
- new net: J2.1 (Pin_1), SW1.2 (B)
- no-connect marks 22 -> 23
Changed lines of the file:
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@@
 	)
 	(no_connect
+		(at 57.15 54.61)
+	)
+	(no_connect
 		(at 224.79 113.03)
 	)
@@
 	(wire
 		(pts
+			(xy 45.72 52.07) (xy 46.99 52.07)
+		)
+		(stroke
+			(width 0)
+			(type default)
+		)
+	)
+	(wire
+		(pts
 			(xy 38.1 109.22) (xy 40.64 109.22)
 		)
@@
 	(wire
 		(pts
+			(xy 45.72 43.18) (xy 45.72 52.07)
+		)
+		(stroke
+			(width 0)
+			(type default)
+		)
+	)
+	(wire
+		(pts
 			(xy 105.41 60.96) (xy 118.11 60.96)
 		)
@@
 	(wire
 		(pts
-			(xy 261.62 26.67) (xy 261.62 27.94)
+			(xy 57.15 49.53) (xy 58.42 49.53)
 		)
 		(stroke
@@
 	(wire
 		(pts
-			(xy 45.72 43.18) (xy 45.72 44.45)
+			(xy 261.62 26.67) (xy 261.62 27.94)
 		)
 		(stroke
@@
 		)
 	)
-	(label "SD_SCK"
+	(label "SD_CLK"
 		(at 105.41 73.66 0)
 		(effects
@@
 			)
 		)
-		(property "Footprint" ""
+		(property "Footprint" "Connector_PinSocket_2.54mm:PinSocket_1x08_P2.54mm_Vertical"
 			(at 40.64 76.2 0)
 			(hide yes)
@@
 			)
 		)
-		(property "Value" "~"
+		(property "Value" "MicroSD"
 			(at 153.67 133.985 0)
 			(effects
@@
 			)
 		)
-		(property "Footprint" ""
+		(property "Footprint" "Components:MicroSD"
 			(at 143.51 124.46 0)
 			(hide yes)
@@
 	(symbol
 		(lib_id "power:VCC")
-		(at 45.72 44.45 180)
+		(at 58.42 49.53 270)
 		(unit 1)
 		(exclude_from_sim no)
@@
 		(dnp no)
 		(property "Reference" "#PWR01"
-			(at 45.72 40.64 0)
+			(at 54.61 49.53 0)
 			(hide yes)
 			(effects
@@
 		)
 		(property "Value" "VCC"
-			(at 48.514 47.498 0)
+			(at 61.468 46.736 0)
 			(effects
 				(font
@@
 		)
 		(property "Footprint" ""
-			(at 45.72 44.45 0)
+			(at 58.42 49.53 0)
 			(hide yes)
 			(effects
@@
 		)
 		(property "Datasheet" ""
-			(at 45.72 44.45 0)
+			(at 58.42 49.53 0)
 			(hide yes)
 			(effects
@@
 		)
 		(property "Description" "Power symbol creates a global label with name \"VCC\""
-			(at 45.72 44.45 0)
+			(at 58.42 49.53 0)
 			(hide yes)
 			(effects
@@
 	)
 	(symbol
+		(lib_id "Switch:SW_SPDT")
+		(at 52.07 52.07 0)
+		(unit 1)
+		(exclude_from_sim no)
+		(in_bom yes)
+		(on_board yes)
+		(dnp no)
+		(property "Reference" "SW1"
+			(at 52.07 43.18 0)
+			(effects
+				(font
+					(size 1.27 1.27)
+				)
+			)
+		)
+		(property "Value" "SW_SPDT"
+			(at 52.07 45.72 0)
+			(effects
+				(font
+					(size 1.27 1.27)
+				)
+			)
+		)
+		(property "Footprint" "Button_Switch_THT:SW_Slide_SPDT_Angled_CK_OS102011MA1Q"
+			(at 52.07 57.404 0)
+			(hide yes)
+			(effects
+				(font
+					(size 1.27 1.27)
+				)
+			)
+		)
+		(property "Datasheet" "~"
+			(at 52.07 59.69 0)
+			(hide yes)
+			(effects
+				(font
+					(size 1.27 1.27)
+				)
+			)
+		)
+		(property "Description" "Switch, single pole double throw"
+			(at 52.07 52.07 0)
+			(hide yes)
+			(effects
+				(font
+					(size 1.27 1.27)
+				)
+			)
+		)
+		(pin "2"
+		)
+		(pin "3"
+		)
+		(pin "1"
+		)
+		(instances
+			(project ""
+				(path "/3d9d3921-4865-4b24-a190-624ce8e2dfa7"
+					(reference "SW1")
+					(unit 1)
+				)
+			)
+		)
+	)
+	(symbol
 		(lib_id "power:GND")
 		(at 205.74 33.02 270)
@@
 			)
 		)
-		(property "Footprint" ""
+		(property "Footprint" "Connector_PinSocket_2.54mm:PinSocket_1x02_P2.54mm_Vertical"
 			(at 45.72 38.1 0)
 			(hide yes)
@@
 			)
 		)
-		(property "Footprint" ""
+		(property "Footprint" "Components:BMP180"
 			(at 50.8 118.11 0)
 			(hide yes)
