File: Fruit.kicad_sch (KiCad schematic)
At the start: 8 parts, among them IC1 CAM-M8C-0-10, J1 Conn_01x08_Pin, J2 Conn_01x02_Pin, SW1 SW_SPDT, U1 MicroSD, U2 Ai-Thinker-Ra-02, U3 BMP180

Commit message: feat: fully wired PCB
Parts:
- removed U2: Ai-Thinker-Ra-02, RF_Module:Ai-Thinker-Ra-01-LoRa, symbol RF_Module:Ai-Thinker-Ra-02
- added J3: Conn_Coaxial, Connector_Coaxial:SMA_Amphenol_901-143_Horizontal, symbol Connector:Conn_Coaxial
- added U4: Ai-Thinker-Ra-01, RF_Module:Ai-Thinker-Ra-01-LoRa, symbol RF_Module:Ai-Thinker-Ra-01
Connections:
- net +3.3V: now also U4.3 (VDD)
- net GND: now also J3.2 (Ext), U4.16 (GND), U4.2 (GND), U4.9 (GND)
- net LORA_BUSY: now also U4.5 (DIO0)
- net LORA_CS: now also U4.15 (~{NSS})
- net LORA_MISO: now also U4.13 (MISO)
- net LORA_MOSI: now also U4.14 (MOSI)
- net LORA_RESET: now also U4.4 (~{RESET})
- net LORA_SCK: now also U4.12 (SCK)
- new net LORA_ANT: J3.1 (In), U4.1 (ANT)
